File: c64 rom.kicad_sch (KiCad schematic)
At the start: 6 parts, among them U1 27C256

Commit message: Main: Fix Incorrect naming of 5V terminal
Parts:
- VCC1: value VCC -> +5V
Changed lines of the file:
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@@
       (effects (font (size 1.27 1.27)))
     )
-    (property "Value" "VCC" (at 197.485 22.86 0)
+    (property "Value" "+5V" (at 197.485 22.86 0)
       (effects (font (size 1.27 1.27)) hide)
     )
